Commit message: strugle

File: my_r2d2/urdf/r2d2.urdf (robot description, URDF)
Before this commit: robot R2D2, 16 links, 15 joints
Links:
- removed link left_back_wheel
- removed link left_base
- removed link left_front_wheel
- removed link left_gripper
- removed link left_leg
- removed link left_tip
- removed link right_back_wheel
- removed link right_base
- removed link right_front_wheel
- removed link right_gripper
- removed link right_leg
- removed link right_tip
- added link lense; collision cylinder length=0.05 radius=0.03; visual cylinder length=0.05 radius=0.03
- link base_link: mass 10 -> None; geometry collision cylinder length=${bodylen} radius=${width}; visual cylinder length=${bodylen} radius=${width}
- link box: mass 1 -> None
- link gripper_pole: mass 0.05 -> None; geometry collision cylinder length=${polelen} radius=0.01; visual cylinder length=${polelen} radius=0.01
- link head: mass 2 -> None; geometry collision sphere radius=${width}; visual sphere radius=${width}
Joints:
- removed joint base_to_left_leg
- removed joint base_to_right_leg
- removed joint left_back_wheel_joint
- removed joint left_base_joint
- removed joint left_front_wheel_joint
- removed joint left_gripper_joint
- removed joint left_tip_joint
- removed joint right_back_wheel_joint
- removed joint right_base_joint
- removed joint right_front_wheel_joint
- removed joint right_gripper_joint
- removed joint right_tip_joint
- added joint lenjoint: type fixed, parent box, child lense
- joint gripper_extension: limit lower=-0.38 upper=0 effort=1000.0 velocity=0.5 -> lower=-${width*2-.02} upper=0 effort=1000.0 velocity=0.5; origin xyz=0.19 0 0.2 rpy=0 0 0 -> xyz=${width-.01} 0 0.2 rpy=0 0 0
- joint head_swivel: origin xyz=0 0 0.3 -> xyz=0 0 ${bodylen/2}
- joint tobox: origin xyz=0.1814 0 0.1414 -> xyz=${.707*width+0.04} 0 ${.707*width}

Commit message: admamvf

File: my_r2d2/urdf/r2d2.urdf (robot description, URDF)
Before this commit: robot macroed, 5 links, 4 joints
Links:
- added link base_footprint
- link box: geometry collision box size=0.08 0.08 0.08; visual box size=${boxlen} ${boxlen} ${boxlen}
- link lense: geometry collision cylinder length=0.05 radius=0.03; visual cylinder length=${boxlen/4} radius=0.03
Joints:
- added joint footprint_joint: type fixed, parent base_footprint, child base_link, origin xyz=0 0 ${wheeldiam+0.1+bodylen/2}
- joint lenjoint: origin (none) -> xyz=0 0 0 rpy=0 ${pi/2} 0

Commit message: hejke

File: my_r2d2/urdf/r2d2.urdf (robot description, URDF)
Before this commit: robot macroed, 6 links, 5 joints
Links:
- link base_link: geometry collision cylinder length=${bodylen} radius=${width}; visual origin xyz=0 0 0
