Commit message: adf

File: src/my_r2d2/urdf/r2d2.urdf.xacro (robot description, xacro)
@@ -214,4 +214,10 @@
     <origin xyz="${.707*width+0.04} 0 ${.707*width}"/>
   </joint>
+  <link name="eye"/>
+  <joint name="eye_joint" type="fixed">
+    <parent link="lense"/>
+    <child link="eye"/>
+    <origin rpy="${pi/2} ${pi} ${pi/2}"/>
+  </joint>
   <link name="lense">
     <visual>
